File: hp-floppy-debug.kicad_sch (KiCad schematic)
At the start: 74 parts, among them J1 34-Pin HD Floppy Interface, J2 34-Pin HD Floppy Interface, J3 34-Pin HD Floppy Interface, J4 Conn_01x04, J5 Conn_01x05, J6 Conn_01x04, J7 Conn_02x02_Odd_Even, M1 3.5in_HDD_Mount, SW1 RotaryEncoder_Switch, U1 74LS09, U2 74LS09, U3 74LS09, U4 MAX232

Commit message: review changes
Parts:
- added J8: Conn_01x05, Connector_PinHeader_2.54mm:PinHeader_1x05_P2.54mm_Vertical, symbol Connector_Generic:Conn_01x05
- added JP36, JP37, JP38: SolderJumper_2_Bridged, Jumper:SolderJumper-2_P1.3mm_Bridged_RoundedPad1.0x1.5mm, symbol Jumper:SolderJumper_2_Bridged
Connections:
- net DIR: now also JP37.2 (B)
- net DISK_CHANGE: now also JP38.2 (B)
- net GND: now also J8.4 (Pin_4), J8.5 (Pin_5)
- net STEP: now also JP36.2 (B)
- net at A1.12 (D9), J5.2 (Pin_2), SW1.A: now also J8.2 (Pin_2)
- net at A1.11 (D8), J5.3 (Pin_3), SW1.B: now also J8.3 (Pin_3)
- net at A1.13 (D10), J5.1 (Pin_1), SW1.S1: now also J8.1 (Pin_1)
- net at A1.10 (D7): now also JP38.1 (A)
- net at A1.21 (A2): now also JP36.1 (A)
- net at A1.22 (A3): now also JP37.1 (A)
Other:
- moved on the sheet: J5
Changed lines of the file:
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@@
   (junction (at 275.59 156.21) (diameter 0) (color 0 0 0 0)
   )
+  (junction (at 43.18 185.42) (diameter 0) (color 0 0 0 0)
+  )
   (junction (at 17.78 82.55) (diameter 0) (color 0 0 0 0)
   )
@@
   (junction (at 187.96 60.96) (diameter 0) (color 0 0 0 0)
   )
+  (junction (at 43.18 182.88) (diameter 0) (color 0 0 0 0)
+  )
   (junction (at 162.56 114.3) (diameter 0) (color 0 0 0 0)
   )
@@
   (junction (at 187.96 53.34) (diameter 0) (color 0 0 0 0)
   )
+  (junction (at 43.18 180.34) (diameter 0) (color 0 0 0 0)
+  )
   (junction (at 187.96 63.5) (diameter 0) (color 0 0 0 0)
   )
@@
   (junction (at 35.56 187.96) (diameter 0) (color 0 0 0 0)
   )
+  (junction (at 43.18 190.5) (diameter 0) (color 0 0 0 0)
+  )
   (junction (at 25.4 187.96) (diameter 0) (color 0 0 0 0)
   )
@@
     (stroke (width 0) (type default) (color 0 0 0 0))
   )
+  (wire (pts (xy 58.42 190.5) (xy 43.18 190.5))
+    (stroke (width 0) (type default) (color 0 0 0 0))
+  )
   (wire (pts (xy 129.54 33.02) (xy 151.13 33.02))
     (stroke (width 0) (type default) (color 0 0 0 0))
@@
     (stroke (width 0) (type default) (color 0 0 0 0))
   )
+  (wire (pts (xy 58.42 187.96) (xy 43.18 187.96))
+    (stroke (width 0) (type default) (color 0 0 0 0))
+  )
   (wire (pts (xy 275.59 120.65) (xy 275.59 123.19))
     (stroke (width 0) (type default) (color 0 0 0 0))
@@
     (stroke (width 0) (type default) (color 0 0 0 0))
   )
+  (wire (pts (xy 58.42 185.42) (xy 43.18 185.42))
+    (stroke (width 0) (type default) (color 0 0 0 0))
+  )
   (wire (pts (xy 16.51 146.05) (xy 33.02 146.05))
     (stroke (width 0) (type default) (color 0 0 0 0))
@@
     (stroke (width 0) (type default) (color 0 0 0 0))
   )
+  (wire (pts (xy 58.42 180.34) (xy 43.18 180.34))
+    (stroke (width 0) (type default) (color 0 0 0 0))
+  )
   (wire (pts (xy 243.84 156.21) (xy 251.46 156.21))
     (stroke (width 0) (type default) (color 0 0 0 0))
@@
     (stroke (width 0) (type default) (color 0 0 0 0))
   )
+  (wire (pts (xy 58.42 182.88) (xy 43.18 182.88))
+    (stroke (width 0) (type default) (color 0 0 0 0))
+  )
   (wire (pts (xy 154.94 129.54) (xy 147.32 129.54))
     (stroke (width 0) (type default) (color 0 0 0 0))
@@
     (effects (font (size 1.27 1.27)) (justify right bottom))
   )
+  (label "STEP" (at 66.04 148.59 0)
+    (effects (font (size 1.27 1.27)) (justify left bottom))
+  )
   (label "RX_EIA" (at 147.32 165.1 0)
     (effects (font (size 1.27 1.27)) (justify left bottom))
@@
     (effects (font (size 1.27 1.27)) (justify right bottom))
   )
+  (label "DISK_CHANGE" (at 25.4 143.51 180)
+    (effects (font (size 1.27 1.27)) (justify right bottom))
+  )
   (label "DS3" (at 33.02 133.35 180)
     (effects (font (size 1.27 1.27)) (justify right bottom))
@@
     (effects (font (size 1.27 1.27)) (justify right bottom))
   )
+  (label "DIR" (at 66.04 151.13 0)
+    (effects (font (size 1.27 1.27)) (justify left bottom))
+  )
   (label "BETA ENABLE" (at 204.47 57.15 180)
     (effects (font (size 1.27 1.27)) (justify right bottom))
@@
     (pin "4")
   )
+  (symbol (lib_id "Jumper:SolderJumper_2_Bridged") (at 29.21 143.51 0) (mirror y) (unit 1)
+    (in_bom yes) (on_board yes)
+    (property "Reference" "JP38" (id 0) (at 26.67 142.24 0))
+    (property "Value" "SolderJumper_2_Bridged" (id 1) (at 29.21 139.7 0)
+      (effects (font (size 1.27 1.27)) hide)
+    )
+    (property "Footprint" "Jumper:SolderJumper-2_P1.3mm_Bridged_RoundedPad1.0x1.5mm" (id 2) (at 29.21 143.51 0)
+      (effects (font (size 1.27 1.27)) hide)
+    )
+    (property "Datasheet" "~" (id 3) (at 29.21 143.51 0)
+      (effects (font (size 1.27 1.27)) hide)
+    )
+    (pin "1")
+    (pin "2")
+  )
   (symbol (lib_id "Jumper:SolderJumper_2_Bridged") (at 58.42 87.63 0) (unit 1)
     (in_bom yes) (on_board yes)
@@
     (pin "2")
   )
+  (symbol (lib_id "Jumper:SolderJumper_2_Bridged") (at 62.23 148.59 0) (unit 1)
+    (in_bom yes) (on_board yes)
+    (property "Reference" "JP36" (id 0) (at 64.77 147.32 0))
+    (property "Value" "SolderJumper_2_Bridged" (id 1) (at 62.23 144.78 0)
+      (effects (font (size 1.27 1.27)) hide)
+    )
+    (property "Footprint" "Jumper:SolderJumper-2_P1.3mm_Bridged_RoundedPad1.0x1.5mm" (id 2) (at 62.23 148.59 0)
+      (effects (font (size 1.27 1.27)) hide)
+    )
+    (property "Datasheet" "~" (id 3) (at 62.23 148.59 0)
+      (effects (font (size 1.27 1.27)) hide)
+    )
+    (pin "1")
+    (pin "2")
+  )
   (symbol (lib_id "Jumper:SolderJumper_2_Bridged") (at 222.25 128.27 0) (mirror y) (unit 1)
     (in_bom yes) (on_board yes)
@@
     (pin "1")
   )
-  (symbol (lib_id "Connector_Generic:Conn_01x05") (at 48.26 185.42 0) (unit 1)
+  (symbol (lib_id "Connector_Generic:Conn_01x05") (at 63.5 185.42 0) (unit 1)
     (in_bom yes) (on_board yes) (fields_autoplaced)
-    (property "Reference" "J5" (id 0) (at 50.8 184.1499 0)
+    (property "Reference" "J5" (id 0) (at 66.04 184.1499 0)
       (effects (font (size 1.27 1.27)) (justify left))
     )
-    (property "Value" "Conn_01x05" (id 1) (at 50.8 186.6899 0)
+    (property "Value" "Conn_01x05" (id 1) (at 66.04 186.6899 0)
       (effects (font (size 1.27 1.27)) (justify left))
     )
-    (property "Footprint" "Connector_PinHeader_2.54mm:PinHeader_1x05_P2.54mm_Vertical" (id 2) (at 48.26 185.42 0)
+    (property "Footprint" "Connector_PinHeader_2.54mm:PinHeader_1x05_P2.54mm_Vertical" (id 2) (at 63.5 185.42 0)
       (effects (font (size 1.27 1.27)) hide)
     )
-    (property "Datasheet" "~" (id 3) (at 48.26 185.42 0)
+    (property "Datasheet" "~" (id 3) (at 63.5 185.42 0)
       (effects (font (size 1.27 1.27)) hide)
     )
@@
     (pin "7")
   )
+  (symbol (lib_id "Connector_Generic:Conn_01x05") (at 48.26 185.42 0) (unit 1)
+    (in_bom yes) (on_board yes) (fields_autoplaced)
+    (property "Reference" "J8" (id 0) (at 50.8 184.1499 0)
+      (effects (font (size 1.27 1.27)) (justify left))
+    )
+    (property "Value" "Conn_01x05" (id 1) (at 50.8 186.6899 0)
+      (effects (font (size 1.27 1.27)) (justify left))
+    )
+    (property "Footprint" "Connector_PinHeader_2.54mm:PinHeader_1x05_P2.54mm_Vertical" (id 2) (at 48.26 185.42 0)
+      (effects (font (size 1.27 1.27)) hide)
+    )
+    (property "Datasheet" "~" (id 3) (at 48.26 185.42 0)
+      (effects (font (size 1.27 1.27)) hide)
+    )
+    (pin "1")
+    (pin "2")
+    (pin "3")
+    (pin "4")
+    (pin "5")
+  )
   (symbol (lib_id "Jumper:SolderJumper_2_Bridged") (at 58.42 100.33 0) (unit 1)
     (in_bom yes) (on_board yes)
@@
     (pin "1")
   )
+  (symbol (lib_id "Jumper:SolderJumper_2_Bridged") (at 62.23 151.13 0) (unit 1)
+    (in_bom yes) (on_board yes)
+    (property "Reference" "JP37" (id 0) (at 64.77 149.86 0))
+    (property "Value" "SolderJumper_2_Bridged" (id 1) (at 62.23 147.32 0)
+      (effects (font (size 1.27 1.27)) hide)
+    )
+    (property "Footprint" "Jumper:SolderJumper-2_P1.3mm_Bridged_RoundedPad1.0x1.5mm" (id 2) (at 62.23 151.13 0)
+      (effects (font (size 1.27 1.27)) hide)
+    )
+    (property "Datasheet" "~" (id 3) (at 62.23 151.13 0)
+      (effects (font (size 1.27 1.27)) hide)
+    )
+    (pin "1")
+    (pin "2")
+  )
   (symbol (lib_id "power:+5V") (at 64.77 19.05 0) (unit 1)
     (in_bom yes) (on_board yes) (fields_autoplaced)
@@
       (reference "J7") (unit 1) (value "Conn_02x02_Odd_Even") (footprint "Connector_PinHeader_2.54mm:PinHeader_2x02_P2.54mm_Vertical")
     )
+    (path "/8ba6e762-dfea-495f-9a52-913479f3bd21"
+      (reference "J8") (unit 1) (value "Conn_01x05") (footprint "Connector_PinHeader_2.54mm:PinHeader_1x05_P2.54mm_Vertical")
+    )
     (path "/8231b19c-ae8e-483e-8754-7633ede6e6be"
       (reference "JP1") (unit 1) (value "SolderJumper_2_Bridged") (footprint "Jumper:SolderJumper-2_P1.3mm_Bridged_RoundedPad1.0x1.5mm")
@@
       (reference "JP35") (unit 1) (value "SolderJumper_2_Bridged") (footprint "Jumper:SolderJumper-2_P1.3mm_Bridged_RoundedPad1.0x1.5mm")
     )
+    (path "/66cdba15-5f57-49f3-a69b-06f8ffb7ac1b"
+      (reference "JP36") (unit 1) (value "SolderJumper_2_Bridged") (footprint "Jumper:SolderJumper-2_P1.3mm_Bridged_RoundedPad1.0x1.5mm")
+    )
+    (path "/9f58e785-600e-4270-9ea3-8a32de97511b"
+      (reference "JP37") (unit 1) (value "SolderJumper_2_Bridged") (footprint "Jumper:SolderJumper-2_P1.3mm_Bridged_RoundedPad1.0x1.5mm")
+    )
+    (path "/1dad116a-861a-46d6-93fb-9b6a8848d819"
+      (reference "JP38") (unit 1) (value "SolderJumper_2_Bridged") (footprint "Jumper:SolderJumper-2_P1.3mm_Bridged_RoundedPad1.0x1.5mm")
+    )
     (path "/41920cd9-afbc-4ad7-8514-dac67dc83462"
